File: PCB/ownly-top-plate.kicad_pcb (KiCad board)
At the start: 2 copper layers, 254.8 x 110.7 mm, 63 parts

Commit message: 製品版をコミット
Parts:
- removed the REF** at (177.5, 129.5)
- removed the REF** at (169.1, 67.3)
- removed the REF** at (150.0, 67.3)
- removed the REF** at (188.1, 67.3)
- removed the REF** at (240.5, 124.4)
- removed the REF** at (221.5, 124.4)
- removed the REF** at (259.6, 124.4)
- removed the REF** at (259.6, 105.4)
- removed the REF** at (240.5, 105.4)
- removed the REF** at (221.5, 105.4)
- removed the REF** at (202.4, 105.4)
- removed the REF** at (201.0, 125.8)
- removed the REF** at (183.4, 105.4)
- removed the REF** at (164.3, 105.4)
- removed the REF** at (235.7, 48.2)
- removed the REF** at (216.7, 48.2)
- removed the REF** at (197.6, 48.2)
- removed the REF** at (178.6, 48.2)
- removed the REF** at (159.5, 48.2)
- removed the REF** at (140.5, 48.2)
- removed the REF** at (139.3, 135.1)
- removed the REF** at (111.6, 128.2)
- removed the REF** at (254.8, 48.2)
- removed the REF** at (211.9, 86.3)
- removed the REF** at (31.0, 88.1)
- removed the REF** at (226.2, 67.3)
- removed the REF** at (207.2, 67.3)
- removed the REF** at (173.8, 86.3)
- removed the REF** at (154.8, 86.3)
- removed the REF** at (192.9, 86.3)
- removed Ref101: Val1, kbd:M2_HOLE
- removed Ref102: Val2, kbd:M2_HOLE
- removed Ref103: Val3, kbd:M2_HOLE
- removed Ref105: Val5, kbd:M2_HOLE
- removed Ref106: Val6, kbd:M2_HOLE
- removed Ref107: Val7, kbd:M2_HOLE
- removed Ref108: Val8, kbd:M2_HOLE
- added REF**: MountingHole_2.2mm_M2, MountingHole:MountingHole_2.2mm_M2, F.Cu at (266.1, 55.8)
- added REF**: MountingHole_2.2mm_M2, MountingHole:MountingHole_2.2mm_M2, F.Cu at (19.4, 145.0)
- added REF**: MountingHole_2.2mm_M2, MountingHole:MountingHole_2.2mm_M2, F.Cu at (238.1, 56.4)
- added REF**: SW_PUSH, keyboard:Switch_Cuts, F.Cu at (195.0, 84.1)
- added REF**: SW_PUSH, keyboard:Switch_Cuts, F.Cu at (156.9, 84.1)
- added REF**: SW_PUSH, keyboard:Switch_Cuts, F.Cu at (214.0, 84.1)
- added REF**: SW_PUSH, keyboard:Switch_Cuts, F.Cu at (233.1, 84.1)
- added REF**: SW_PUSH, keyboard:Switch_Cuts, F.Cu at (175.9, 84.1)
- added REF**: SW_PUSH, keyboard:Switch_Cuts, F.Cu at (203.2, 123.5)
- added REF**: plate-stabilizer, locallib:plate-stabilizer, F.Cu at (171.9, 130.5)
- added REF**: SW_PUSH, keyboard:Switch_Cuts, F.Cu at (261.6, 122.2)
- added REF**: MountingHole_2.2mm_M2, MountingHole:MountingHole_2.2mm_M2, F.Cu at (160.3, 117.3)
- added REF**: SW_PUSH, keyboard:Switch_Cuts, F.Cu at (223.5, 122.2)
- added REF**: SW_PUSH, keyboard:Switch_Cuts, F.Cu at (242.6, 122.2)
- added REF**: SW_PUSH, keyboard:Switch_Cuts, F.Cu at (204.5, 103.1)
- added REF**: SW_PUSH, keyboard:Switch_Cuts, F.Cu at (242.6, 103.1)
- added REF**: SW_PUSH, keyboard:Switch_Cuts, F.Cu at (166.4, 103.1)
- added REF**: SW_PUSH, keyboard:Switch_Cuts, F.Cu at (185.4, 103.1)
- added REF**: SW_PUSH, keyboard:Switch_Cuts, F.Cu at (261.6, 103.1)
- added REF**: SW_PUSH, keyboard:Switch_Cuts, F.Cu at (223.5, 103.1)
- added REF**: SW_PUSH, keyboard:Switch_Cuts, F.Cu at (190.2, 65.0)
- added REF**: SW_PUSH, keyboard:Switch_Cuts, F.Cu at (228.3, 65.0)
- added REF**: MountingHole_2.2mm_M2, MountingHole:MountingHole_2.2mm_M2, F.Cu at (191.4, 140.9)
- added REF**: SW_PUSH, keyboard:Switch_Cuts, F.Cu at (152.1, 65.0)
- added REF**: SW_PUSH, keyboard:Switch_Cuts, F.Cu at (171.2, 65.0)
- added REF**: SW_PUSH, keyboard:Switch_Cuts, F.Cu at (209.3, 65.0)
- added REF**: MountingHole_2.2mm_M2, MountingHole:MountingHole_2.2mm_M2, F.Cu at (162.8, 56.4)
- added REF**: SW_PUSH, keyboard:Switch_Cuts, F.Cu at (256.9, 46.0)
- added REF**: SW_PUSH, keyboard:Switch_Cuts, F.Cu at (237.8, 46.0)
- added REF**: SW_PUSH, keyboard:Switch_Cuts, F.Cu at (142.6, 46.0)
- added REF**: SW_PUSH, keyboard:Switch_Cuts, F.Cu at (218.8, 46.0)
- added REF**: SW_PUSH, keyboard:Switch_Cuts, F.Cu at (161.6, 46.0)
- added REF**: SW_PUSH, keyboard:Switch_Cuts, F.Cu at (180.7, 46.0)
- added REF**: MountingHole_2.2mm_M2, MountingHole:MountingHole_2.2mm_M2, F.Cu at (266.1, 140.9)
- added REF**: SW_PUSH, keyboard:Switch_Cuts, F.Cu at (199.7, 46.0)
- added REF**: plate-stabilizer, locallib:plate-stabilizer, F.Cu at (123.2, 133.1)
- added REF**: SW_PUSH, keyboard:Switch_Cuts, F.Cu at (94.0, 127.3)
- added REF**: SW_PUSH, keyboard:Switch_Cuts, F.Cu at (71.4, 126.2)
- added REF**: MountingHole_2.2mm_M2, MountingHole:MountingHole_2.2mm_M2, F.Cu at (95.3, 97.6)
- added REF**: SW_PUSH, keyboard:Switch_Cuts_1.75u, F.Cu at (31.0, 88.1)
- added REF**: MountingHole_2.2mm_M2, MountingHole:MountingHole_2.2mm_M2, F.Cu at (61.9, 59.5)
- added REF**: MountingHole_2.2mm_M2, MountingHole:MountingHole_2.2mm_M2, F.Cu at (118.8, 60.4)
- added REF**: MountingHole_2.2mm_M2, MountingHole:MountingHole_2.2mm_M2, F.Cu at (19.4, 61.8)
- added REF**: MountingHole_2.2mm_M2, MountingHole:MountingHole_2.2mm_M2, F.Cu at (144.4, 121.3)
- added REF**: MountingHole_2.2mm_M2, MountingHole:MountingHole_2.2mm_M2, F.Cu at (100.5, 145.0)
- moved G*** 8.64 mm to (50.9, 140.6)
- moved G*** 4.84 mm to (249.0, 137.7)
Other:
- board size 254.8 x 110.7 mm -> 256.9 x 113.6 mm
- board text added: "ownly rev2.0.0 PCB designed by Diwamoto"
- board text removed: "ownly58 rev1.0.0 PCB designed by Diwamoto for gaming ,coding, typing, etc..."
