File: PCB/ownly.kicad_pcb (KiCad board)
At the start: 2 copper layers, 254.8 x 132.2 mm, 220 parts, among them J1 OLED, J2 i2c_pin, J3 i2c_pin, J4 MJ-4PP-9, J5 OLED, J6 MJ-4PP-9, J7 i2c_pin, J8 i2c_pin, SW1 SW_PUSH, SW10 SW_PUSH, SW11 SW_PUSH, SW12 SW_PUSH, SW13 SW_PUSH, SW14 SW_PUSH, SW15 SW_PUSH, SW16 SW_PUSH, SW17 SW_PUSH, SW18 SW_PUSH, SW19 SW_PUSH, SW2 SW_PUSH, SW20 SW_PUSH, SW21 SW_PUSH, SW22 SW_PUSH, SW23 SW_PUSH, SW24 SW_PUSH, SW25 SW_PUSH, SW26 SW_PUSH, SW27 SW_PUSH, SW28 SW_PUSH, SW29 SW_PUSH, SW3 SW_PUSH, SW30 SW_PUSH, SW31 SW_PUSH, SW32 SW_PUSH, SW33 SW_PUSH, SW34 SW_PUSH, SW35 SW_PUSH, SW36 SW_PUSH, SW37 SW_PUSH, SW38 SW_PUSH, SW39 SW_PUSH, SW4 SW_PUSH, SW40 SW_PUSH, SW41 SW_PUSH, SW41' SW_PUSH, SW42 SW_PUSH, SW43 SW_PUSH, SW44 SW_PUSH, SW45 SW_PUSH, SW46 SW_PUSH, SW47 SW_PUSH, SW47' KEY_SWITCH, SW48 SW_PUSH, SW49 SW_PUSH, SW5 SW_PUSH, SW50 SW_PUSH, SW51 SW_PUSH, SW52 SW_PUSH, SW53 SW_PUSH, SW54 SW_PUSH, SW55 SW_PUSH, SW56 SW_PUSH, SW57 SW_PUSH, SW58 SW_PUSH, SW6 SW_PUSH, SW7 SW_PUSH, SW8 SW_PUSH, SW9 SW_PUSH, U1 ProMicro, U2 ProMicro

Commit message: 製品版をコミット
Parts:
- removed D29: D, kbd:D3_SMD
- removed J3, J7, J8: i2c_pin, kbd:1pin_conn
- removed J6: MJ-4PP-9, kbd:MJ-4PP-9_1side
- removed JP1, JP6: Jumper, kbd:JPC2
- removed JP10, JP2, JP3, JP4, JP5, JP7, JP8, JP9: Jumper_NC_Small, kbd:Jumper
- removed L29: YS-SK6812MINI-E, keyboard:YS-SK6812MINI-E
- removed R1, R2, R3, R4: R, kbd:R
- removed REF1, REF2, REF7, REF8: MountingHole_2.2mm_M2, MountingHole:MountingHole_2.2mm_M2
- removed Ref103: Val3, kbd:M2_HOLE
- removed the Ref104 at (250.0, 114.6)
- removed Ref105: Val5, kbd:M2_HOLE
- removed Ref106: Val6, kbd:M2_HOLE
- removed the Ref107 at (53.9, 112.5)
- removed SW29: SW_PUSH, kbd:CherryMX_Hotswap_2u
- added Ref104: Val4, kbd:M2_HOLE, F.Cu at (195.0, 93.8)
- added Ref104: Val4, kbd:M2_HOLE, F.Cu at (218.8, 55.8)
- added Ref104: Val4, kbd:M2_HOLE, F.Cu at (191.2, 140.9)
- added Ref104: Val4, kbd:M2_HOLE, F.Cu at (266.0, 55.8)
- added Ref104: Val4, kbd:M2_HOLE, F.Cu at (266.0, 140.9)
- added Ref107: Val7, kbd:M2_HOLE, F.Cu at (19.3, 145.0)
- added Ref107: Val7, kbd:M2_HOLE, F.Cu at (100.5, 145.0)
- added Ref107: Val7, kbd:M2_HOLE, F.Cu at (62.1, 59.5)
- added Ref107: Val7, kbd:M2_HOLE, F.Cu at (95.2, 97.8)
- J2: value i2c_pin -> MJ-4PP-9; footprint kbd:1pin_conn -> kbd:MJ-4PP-9_1side
- SW26: footprint kbd:CherryMX_Hotswap -> kbd:CherryMX_Hotswap_1.25u
- SW28: footprint kbd:CherryMX_Hotswap -> kbd:CherryMX_Hotswap_2u
- SW47': footprint kbd:CherryMX_Hotswap_2u -> kbd:CherryMX_Hotswap_iso_enter
- SW54: footprint kbd:CherryMX_Hotswap_1.5u -> kbd:CherryMX_Hotswap_2.25u
- moved J2 32.8 mm to (144.2, 15.6)
- moved Ref108 23.3 mm to (19.3, 61.8)
- moved L28 12.8 mm to (124.5, 128.3)
- moved SW28 12.6 mm to (123.2, 133.1)
- moved G*** 7.96 mm to (50.2, 139.2)
- moved L54 6.11 mm to (170.7, 125.6), turned to 15 degrees
- moved SW54 5.71 mm to (171.9, 130.5), turned to 195 degrees
- moved D54 5.46 mm to (163.0, 126.1)
- moved D28 5.36 mm to (108.9, 126.2)
- moved G*** 4.53 mm to (247.4, 136.9)
- moved L27 4.25 mm to (94.6, 122.2), turned to 353.5 degrees
- moved SW27 3.66 mm to (94.0, 127.3), turned to 173.5 degrees
- moved L55 3.34 mm to (202.5, 118.3), turned to 7.5 degrees
- moved SW55 3.23 mm to (203.2, 123.5), turned to 187.5 degrees
- moved Ref102 3.11 mm to (161.6, 55.7)
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Connections:
- J1 pad 1: Net-(J1-Pad1) -> SDA2
- J1 pad 2: Net-(J1-Pad2) -> SCL2
- J1 pad 3: Net-(J1-Pad3) -> VCC
- J1 pad 4: Net-(J1-Pad4) -> GND
- J4 pad A: Net-(J2-Pad1) -> Net-(J4-PadA)
- J4 pad B: Net-(J3-Pad1) -> data1
- J5 pad 1: Net-(J5-Pad1) -> SDA1
- J5 pad 2: Net-(J5-Pad2) -> SCL1
- J5 pad 3: Net-(J5-Pad3) -> VCC
- J5 pad 4: Net-(J5-Pad4) -> GND
- L24 pad 4: Net-(L24-Pad4) -> LED1
- SW41' pad 2: Net-(D35-Pad2) -> Net-(D41-Pad2)
Routing:
- net GND: track 1629.7 -> 1517.2 mm
- net row4: track 250.6 -> 214.1 mm, vias 2 -> 6
- net Net-(D41-Pad2): track 4.44 -> 39.4 mm, vias 0 -> 2
- net VCC: track 1423.8 -> 1389.0 mm, vias 31 -> 33
- net col5: track 134.6 -> 103.2 mm
- net Net-(L24-Pad4): track 31.3 -> 0.00 mm, vias 2 -> 0
- net Net-(D35-Pad2): track 35.2 -> 4.86 mm, vias 4 -> 0
- net Net-(J3-Pad1): track 26.5 -> 0.00 mm, vias 1 -> 0
- net Net-(J6-PadB): track 23.2 -> 0.00 mm, vias 2 -> 0
- net LED1: track 149.5 -> 127.2 mm
- net Net-(D29-Pad2): track 15.5 -> 0.00 mm
- net SCL2: track 38.7 -> 24.1 mm, vias 1 -> 0
- net SDA1: track 42.6 -> 30.9 mm, vias 1 -> 0
- net SDA2: track 38.9 -> 27.6 mm, vias 1 -> 0
- net row04: track 216.6 -> 206.6 mm, vias 1 -> 3
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Other:
- board size 254.8 x 132.2 mm -> 256.9 x 135 mm
- board text added: "ownly rev2.0.0 PCB designed by Diwamoto"
- board text removed: "ownly58 rev1.0.0 PCB designed by Diwamoto for gaming ,coding, typing, etc..."
